Commit message: add dummy inertial to links

File: urdf/combined_robot.urdf (robot description, URDF)
Before this commit: robot jacobi_robot, 11 links, 10 joints
Links:
- link abb_arm_base_link: mass None -> 1.0
- link abb_arm_link_1: mass None -> 1.0
- link abb_arm_link_2: mass None -> 1.0
- link abb_arm_link_3: mass None -> 1.0
- link abb_arm_link_4: mass None -> 1.0
- link abb_arm_link_5: mass None -> 1.0
- link abb_arm_link_6: mass None -> 1.0
- link linear_axis_base_link: mass None -> 1.0
- link linear_axis_link_1: mass None -> 1.0
